Commit message: mods trasporting

File: inmoov_arm_v2_2_reaching_BB.urdf (robot description, URDF)
Before this commit: robot inmoov, 9 links, 8 joints
Links:
- link r_forearm_link: geometry collision box size=0.06 0.06 0.2; visual mesh filename=package://inmoov_meshes/meshes/r_forearm.stl scale=0.001 0.001 0.001
Joints:
- joint r_shoulder_lift_joint: limit lower=-1.57079632679 upper=1.57079632679 effort=1000.0 velocity=1745.32925199 -> lower=-2.07079632679 upper=1.57079632679 effort=1000.0 velocity=1745.32925199
- joint r_shoulder_out_joint: limit lower=-1.57079632679 upper=1.57079632679 effort=1000.0 velocity=1745.32925199 -> lower=-2.07079632679 upper=1.57079632679 effort=1000.0 velocity=1745.32925199
