Commit message: make moving hand BB larger etc.

File: inmoov_arm_v2_2_moving_BB.urdf (robot description, URDF)
Before this commit: robot inmoov, 9 links, 8 joints
Links:
- link rh_palm: geometry collision box size=0.12 0.12 0.15; visual box size=0.12 0.12 0.15

Commit message: combine move and reach code, some hacks

File: inmoov_arm_v2_2_moving_BB.urdf (robot description, URDF)
Before this commit: robot inmoov, 9 links, 8 joints
Links:
- link rh_palm: geometry collision box size=0.18 0.15 0.18; visual box size=0.18 0.15 0.18

File: inmoov_arm_v2_2_reaching_BB.urdf (robot description, URDF)
Before this commit: robot inmoov, 9 links, 8 joints
Links:
- link r_forearm_link: geometry collision box size=0.04 0.04 0.22; visual mesh filename=package://inmoov_meshes/meshes/r_forearm.stl scale=0.001 0.001 0.001
- link rh_palm: geometry collision box size=0.10 0.10 0.18; visual box size=0.10 0.10 0.18

Commit message: minor mods

File: inmoov_arm_v2_2_moving_BB.urdf (robot description, URDF)
Before this commit: robot inmoov, 9 links, 8 joints
Links:
- link rh_palm: geometry collision box size=0.18 0.15 0.18; visual box size=0.15 0.15 0.18

File: inmoov_arm_v2_2_reaching_BB.urdf (robot description, URDF)
Before this commit: robot inmoov, 9 links, 8 joints
Links:
- link rh_palm: geometry collision box size=0.10 0.10 0.18; visual box size=0.15 0.15 0.18

Commit message: fixes reach tabletop odd

File: inmoov_arm_v2_2_moving_BB.urdf (robot description, URDF)
Before this commit: robot inmoov, 9 links, 8 joints
Links:
- link rh_palm: geometry collision box size=0.18 0.15 0.18

File: inmoov_arm_v2_2_reaching_BB.urdf (robot description, URDF)
Before this commit: robot inmoov, 9 links, 8 joints
Links:
- link r_forearm_link: geometry collision box size=0.07 0.07 0.22; visual mesh filename=package://inmoov_meshes/meshes/r_forearm.stl scale=0.001 0.001 0.001
- link rh_palm: geometry collision box size=0.10 0.10 0.18

Commit message: update urdf for openrave viz

File: inmoov_arm_v2_2_moving_BB.urdf (robot description, URDF)
Before this commit: robot inmoov, 9 links, 8 joints
Links:
- link r_forearm_link: geometry collision box size=0.07 0.07 0.2; visual mesh filename=package://inmoov_meshes/meshes/box-binary.stl scale=0.07 0.07 0.2
- link rh_palm: geometry collision box size=0.18 0.15 0.18; visual mesh filename=package://inmoov_meshes/meshes/box-binary.stl scale=0.18 0.15 0.18
- link rh_wrist: geometry visual mesh filename=package://sr_description/hand/model/wrist.dae scale=0.001 0.001 0.001

File: inmoov_arm_v2_2_reaching_BB.urdf (robot description, URDF)
Before this commit: robot inmoov, 9 links, 8 joints
Links:
- link r_forearm_link: geometry collision box size=0.07 0.07 0.2; visual mesh filename=package://inmoov_meshes/meshes/box-binary.stl scale=0.07 0.07 0.2
- link rh_palm: geometry collision box size=0.10 0.10 0.18; visual mesh filename=package://inmoov_meshes/meshes/box-binary.stl scale=0.10 0.10 0.18
- link rh_wrist: geometry visual mesh filename=package://sr_description/hand/model/wrist.dae scale=0.001 0.001 0.001

Commit message: reaching parabolic

File: inmoov_arm_v2_2_moving_BB.urdf (robot description, URDF)
Before this commit: robot inmoov, 9 links, 8 joints
Joints:
- joint r_elbow_flex_joint: limit lower=-3.14159265359 upper=0.0 effort=1000.0 velocity=1745.32925199 -> lower=-3.14159265359 upper=0.0 effort=1000.0 velocity=1
- joint r_elbow_roll_joint: limit lower=-1.57079632679 upper=1.57079632679 effort=1000.0 velocity=1745.32925199 -> lower=-1.57079632679 upper=1.57079632679 effort=1000.0 velocity=1
- joint r_shoulder_lift_joint: limit lower=-2.07079632679 upper=1.57079632679 effort=1000.0 velocity=1745.32925199 -> lower=-2.07079632679 upper=1.57079632679 effort=1000.0 velocity=1
- joint r_shoulder_out_joint: limit lower=-2.07079632679 upper=1.57079632679 effort=1000.0 velocity=1745.32925199 -> lower=-2.07079632679 upper=1.57079632679 effort=1000.0 velocity=1
- joint r_upper_arm_roll_joint: limit lower=-1.57079632679 upper=1.57079632679 effort=1000.0 velocity=1745.32925199 -> lower=-1.57079632679 upper=1.57079632679 effort=1000.0 velocity=1
- joint rh_WRJ1: limit lower=-1.57079632679 upper=1.57079632679 effort=30 velocity=20.0 -> lower=-1.57079632679 upper=1.57079632679 effort=30 velocity=1
- joint rh_WRJ2: limit lower=-1.0471975512 upper=1.0471975512 effort=10 velocity=20.0 -> lower=-1.0471975512 upper=1.0471975512 effort=10 velocity=1

File: inmoov_arm_v2_2_reaching_BB.urdf (robot description, URDF)
Before this commit: robot inmoov, 9 links, 8 joints
Links:
- link rh_palm: geometry collision box size=0.11 0.11 0.16; visual mesh filename=package://inmoov_meshes/meshes/box-binary.stl scale=0.11 0.11 0.16
Joints:
- joint r_elbow_flex_joint: limit lower=-3.14159265359 upper=0.0 effort=1000.0 velocity=1745.32925199 -> lower=-3.14159265359 upper=0.0 effort=1000.0 velocity=1
- joint r_elbow_roll_joint: limit lower=-1.57079632679 upper=1.57079632679 effort=1000.0 velocity=1745.32925199 -> lower=-1.57079632679 upper=1.57079632679 effort=1000.0 velocity=1
- joint r_shoulder_lift_joint: limit lower=-2.07079632679 upper=1.57079632679 effort=1000.0 velocity=1745.32925199 -> lower=-2.07079632679 upper=1.57079632679 effort=1000.0 velocity=1
- joint r_shoulder_out_joint: limit lower=-2.07079632679 upper=1.57079632679 effort=1000.0 velocity=1745.32925199 -> lower=-2.07079632679 upper=1.57079632679 effort=1000.0 velocity=1
- joint r_upper_arm_roll_joint: limit lower=-1.57079632679 upper=1.57079632679 effort=1000.0 velocity=1745.32925199 -> lower=-1.57079632679 upper=1.57079632679 effort=1000.0 velocity=1
- joint rh_WRJ1: limit lower=-1.57079632679 upper=1.57079632679 effort=30 velocity=20.0 -> lower=-1.57079632679 upper=1.57079632679 effort=30 velocity=1
- joint rh_WRJ2: limit lower=-1.0471975512 upper=1.0471975512 effort=10 velocity=20.0 -> lower=-1.0471975512 upper=1.0471975512 effort=10 velocity=1

Commit message: increase vel limit, need clean up wip

File: inmoov_arm_v2_2_moving_BB.urdf (robot description, URDF)
Before this commit: robot inmoov, 9 links, 8 joints
Joints:
- joint r_elbow_flex_joint: limit lower=-3.14159265359 upper=0.0 effort=1000.0 velocity=1 -> lower=-3.14159265359 upper=0.0 effort=1000.0 velocity=2000
- joint r_elbow_roll_joint: limit lower=-1.57079632679 upper=1.57079632679 effort=1000.0 velocity=1 -> lower=-1.57079632679 upper=1.57079632679 effort=1000.0 velocity=2000
- joint r_shoulder_lift_joint: limit lower=-2.07079632679 upper=1.57079632679 effort=1000.0 velocity=1 -> lower=-2.07079632679 upper=1.57079632679 effort=1000.0 velocity=2000
- joint r_shoulder_out_joint: limit lower=-2.07079632679 upper=1.57079632679 effort=1000.0 velocity=1 -> lower=-2.07079632679 upper=1.57079632679 effort=1000.0 velocity=2000
- joint r_upper_arm_roll_joint: limit lower=-1.57079632679 upper=1.57079632679 effort=1000.0 velocity=1 -> lower=-1.57079632679 upper=1.57079632679 effort=1000.0 velocity=2000
- joint rh_WRJ1: limit lower=-1.57079632679 upper=1.57079632679 effort=30 velocity=1 -> lower=-1.57079632679 upper=1.57079632679 effort=30 velocity=20
- joint rh_WRJ2: limit lower=-1.0471975512 upper=1.0471975512 effort=10 velocity=1 -> lower=-1.0471975512 upper=1.0471975512 effort=10 velocity=20

Commit message: add back retract

File: inmoov_arm_v2_2_moving_BB.urdf (robot description, URDF)
Before this commit: robot inmoov, 9 links, 8 joints
Links:
- link r_forearm_link: geometry collision box size=0.06 0.06 0.2; visual mesh filename=package://inmoov_meshes/meshes/box-binary.stl scale=0.06 0.06 0.2
- link rh_palm: geometry collision box size=0.18 0.13 0.18; visual mesh filename=package://inmoov_meshes/meshes/box-binary.stl scale=0.18 0.15 0.18

File: inmoov_arm_v2_2_reaching_BB.urdf (robot description, URDF)
Before this commit: robot inmoov, 9 links, 8 joints
Links:
- link r_forearm_link: geometry collision box size=0.06 0.06 0.2; visual mesh filename=package://inmoov_meshes/meshes/box-binary.stl scale=0.06 0.06 0.2
